File: OpenBCI.sch (KiCad schematic (older format))
At the start: 62 parts, among them J1 CONN_01X08, J1 MicroSD, J2 CONN_01X02, U1 ADXL345, U3 LM2664, U4 TLV700xx, U5 LP5907, U6 ADS1299

Commit message: + Microcontroller and RFDUINO Module
Parts:
- added BLE1: RFD22301, RFD22301, symbol RFD22301
- added C20, C23: 10pF, symbol C
- added C25: 10uF, symbol C
- added D1: BLUE LED, symbol LED
- added D8: LED, symbol LED
- added R10: 220K, symbol R
- added R11: 330K, symbol R
- added R7, R9: 470K, symbol R
- added R8: 1K, symbol R
- added SW1, SW3: PTS810, symbol PTS810
- added SW2: CUS-13B, symbol CUS-13B
- added U7: PIC32MX250F128B, symbol PIC32MX250F128B
- added X1: 8MHz, symbol QUARTZCMS4
- gave numbers to parts that had none: 3
- renumbered C1 to C16, J1 to CONN1
Connections:
- net labels added: RF_RESET, RF_RXD, RF_TXD, RXD, TXD
- wire segments 438 -> 528
- no-connect marks 18 -> 20
Other:
- note added: "MICROCONTROLLER"
- note added: "RFDUINO MODULE"

Commit message: Some fixes on schematic thanks to the electrical rules checker. ADS1299 library component correction for pin 64.
Connections:
- wire segments 528 -> 530
- no-connect marks 20 -> 26
Changed lines of the file:
@@
 P 8500 5700
 F 0 "#PWR01" H 8500 5450 50  0001 C CNN
-F 1 "GNDA" V 8600 5650 50  0000 C CNN
+F 1 "GNDA" H 8500 5550 50  0000 C CNN
 F 2 "" H 8500 5700 60  0000 C CNN
 F 3 "" H 8500 5700 60  0000 C CNN
@@
 L GNDA #PWR020
 U 1 1 5674D5A5
-P 900 7250
-F 0 "#PWR020" H 900 7000 50  0001 C CNN
-F 1 "GNDA" H 900 7100 50  0000 C CNN
-F 2 "" H 900 7250 50  0000 C CNN
-F 3 "" H 900 7250 50  0000 C CNN
-	1    900  7250
+P 900 7300
+F 0 "#PWR020" H 900 7050 50  0001 C CNN
+F 1 "GNDA" H 900 7150 50  0000 C CNN
+F 2 "" H 900 7300 50  0000 C CNN
+F 3 "" H 900 7300 50  0000 C CNN
+	1    900  7300
 	1    0    0    -1
 $EndComp
@@
 RFDUINO MODULE
 Wire Wire Line
-	8000 6050 7750 6050
-Wire Wire Line
-	8000 6150 7750 6150
-Wire Wire Line
-	8000 6250 7750 6250
-Wire Wire Line
 	8000 6350 7750 6350
 Wire Wire Line
@@
 	10950 2500 11350 2500
 Wire Wire Line
-	10950 2600 11350 2600
-Wire Wire Line
 	10950 2700 11350 2700
 Wire Wire Line
@@
 Wire Notes Line
 	11950 4050 8900 4050
-Wire Wire Line
-	10150 1450 10450 1450
 Wire Wire Line
 	10150 1550 10450 1550
@@
 Wire Wire Line
 	1450 8950 1450 8800
-Wire Wire Line
-	1550 8950 1550 8800
 Connection ~ 1450 8950
 Wire Wire Line
@@
 	2700 11100 2700 3900
 Wire Wire Line
-	14250 8350 14250 8450
-Wire Wire Line
 	13800 7400 13350 7400
 Wire Wire Line
@@
 	15850 1050 12150 1050
 Wire Wire Line
-	8700 5600 8500 5600
-Wire Wire Line
-	8500 5600 8500 5700
-Wire Wire Line
 	4550 4300 4600 4300
 Wire Wire Line
@@
 Wire Wire Line
 	6450 3950 6450 4400
+Wire Wire Line
+	10950 2600 11350 2600
+Connection ~ 3600 2550
+Wire Wire Line
+	10150 1450 10450 1450
+Wire Wire Line
+	14250 8450 14250 8350
+Text Label 13450 7600 0    60   ~ 0
+BOOT_EN
+Wire Wire Line
+	1550 8950 1550 8800
+NoConn ~ 1500 7400
+NoConn ~ 1650 8800
+Wire Wire Line
+	8700 5600 8700 5550
+Wire Wire Line
+	8700 5550 8500 5550
+Wire Wire Line
+	8500 5550 8500 5700
+NoConn ~ 15050 1850
+NoConn ~ 15050 1950
+NoConn ~ 15050 2050
+NoConn ~ 15050 2150
+Wire Wire Line
+	8000 6150 7750 6150
+Wire Wire Line
+	8000 6050 7750 6050
+Wire Wire Line
+	8000 6250 7750 6250
+Wire Wire Line
+	900  7250 900  7300
 $EndSCHEMATC
